File: NXP/lpc178x/lpc1788_som/lpc1788_som.kicad_sch (KiCad schematic)
At the start: 1 part, among them U1 LPC1788FBD208

Commit message: Memory connections
Parts:
- renumbered U1 to U101
Other:
- sheet SRAM_Memory renamed uController Core
- added sheet Jtag and Power (jtag_and_power.kicad_sch)
- sheet uController Core: file SRAM_Memory.kicad_sch -> uController_Core.kicad_sch
Changed lines of the file:
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@@
 		(dnp no)
 		(fields_autoplaced yes)
-		(property "Reference" "U1"
+		(property "Reference" "U101"
 			(at -31.75 96.52 0)
 			(effects
@@
 			(project "lpc1788_som"
 				(path "/0de8293f-04e9-4d63-914d-fafec110604e"
-					(reference "U1")
+					(reference "U101")
 					(unit 3)
 				)
@@
 		(dnp no)
 		(fields_autoplaced yes)
-		(property "Reference" "U1"
+		(property "Reference" "U101"
 			(at -90.17 -76.2 0)
 			(effects
@@
 			(project "lpc1788_som"
 				(path "/0de8293f-04e9-4d63-914d-fafec110604e"
-					(reference "U1")
+					(reference "U101")
 					(unit 1)
 				)
@@
 	)
 	(sheet
-		(at 24.13 59.69)
+		(at 104.14 58.42)
 		(size 71.12 16.51)
 		(stroke
@@
 		)
 		(property "Sheetname" "uC_Memory Interface"
-			(at 25.654 58.674 0)
+			(at 105.664 57.404 0)
 			(effects
 				(font
@@
 		)
 		(property "Sheetfile" "uC_Memory.kicad_sch"
-			(at 24.13 75.5146 0)
+			(at 104.14 74.2446 0)
 			(effects
 				(font
@@
 			(project "lpc1788_som"
 				(path "/0de8293f-04e9-4d63-914d-fafec110604e"
-					(page "2")
+					(page "3")
 				)
 			)
@@
 	)
 	(sheet
-		(at 25.4 90.17)
+		(at 104.14 88.9)
 		(size 69.85 12.7)
 		(fields_autoplaced yes)
@@
 			(color 0 0 0 0.0000)
 		)
-		(property "Sheetname" "SRAM_Memory"
-			(at 25.4 87.5934 0)
+		(property "Sheetname" "uController Core"
+			(at 104.14 86.3234 0)
 			(effects
 				(font
@@
 			)
 		)
-		(property "Sheetfile" "SRAM_Memory.kicad_sch"
-			(at 25.4 103.4546 0)
+		(property "Sheetfile" "uController_Core.kicad_sch"
+			(at 104.14 102.1846 0)
 			(effects
 				(font
@@
 			(project "lpc1788_som"
 				(path "/0de8293f-04e9-4d63-914d-fafec110604e"
-					(page "3")
-				)
-			)
+					(page "2")
+				)
+			)
+		)
+	)
+	(sheet
+		(at 104.14 115.57)
+		(size 57.15 15.24)
+		(fields_autoplaced yes)
+		(stroke
+			(width 0.1524)
+			(type solid)
+		)
+		(fill
+			(color 0 0 0 0.0000)
+		)
+		(property "Sheetname" "Jtag and Power"
+			(at 104.14 112.9934 0)
+			(effects
+				(font
+					(size 5 5)
+					(bold yes)
+				)
+				(justify left bottom)
+			)
+		)
+		(property "Sheetfile" "jtag_and_power.kicad_sch"
+			(at 104.14 131.3946 0)
+			(effects
+				(font
+					(size 1.27 1.27)
+				)
+				(justify left top)
+			)
+		)
+		(instances
+			(project "lpc1788_som"
+				(path "/0de8293f-04e9-4d63-914d-fafec110604e"
+					(page "4")
+				)
+			)

Commit message: Add sodim connector
Parts:
- removed U101: LPC1788FBD208, LPC1788FBD208:QFP50P3000X3000X160-208N, symbol _MCU_NXP_LPC:LPC1788FBD208
Other:
- added sheet Power (Power.kicad_sch)
- added sheet sodim connector (sodim_connector.kicad_sch)
