File: NXP/lpc178x/lpc1788_som/jtag_and_power.kicad_sch (KiCad schematic)
At the start: 14 parts, among them J401 Conn_ARM_JTAG_SWD_10, U401 LPC1788FBD208

Commit message: LPC1788
Added LPC1788 som module
Parts:
- added C1, C2: 27pF, symbol Device:C
- added X1: ~, Local_Footprints:OSC-SMD_L3.2-W1.5, symbol Local_symbols:DST310S
Connections:
- net GND: now also C1.1, C2.1
- net RTCX1: now reaches U401.34 (RTCX1)
- net RTCX1: now also C2.2, X1.2
- net RTCX2: now reaches U401.36 (RTCX2)
- net RTCX2: now also C1.2, X1.1
Other:
- note added: "ADC Reference Voltage"
- note added: "External Oscillator and RTC Clock"
- moved on the sheet: C404, C405, X401
