File: Esp8266/esp-wroom-2-carrier-board/microcontroller.kicad_sch (KiCad schematic)
At the start: 19 parts, among them J1 DF9B-19S-1V69, J2 USB_B_Mini, Q1 MMBT2222A, Q2 MMBT2222A, U1 ESP-WROOM-02, U2 FT231XQ

Commit message: Board Layout
Changed board layout to something smaller
Parts:
- removed J2: USB_B_Mini, User_Footprint:Usb_B_mini_Wurth_65100516121, symbol Connector:USB_B_Mini
- added J3: USB_B_Mini, Connector_USB:USB_Mini-B_Lumberg_2486_01_Horizontal, symbol Connector:USB_B_Mini
Connections:
- net +3.3V: now also J1.13, J1.5, J1.9
- net D+: now also J3.3 (D+)
- net D-: now also J3.2 (D-)
- net GND: now also J1.11, J1.15, J1.7, J3.4 (ID), J3.5 (GND), J3.6 (Shield)
- net IO13: no longer J1.13
- net Vbus: now also J3.1 (VBUS)
Changed lines of the file:
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@@
+	)
+	(junction
+		(at 93.98 135.89)
+		(diameter 0)
+		(color 0 0 0 0)
 	)
 	(junction
@@
 	)
 	(junction
-		(at 93.98 135.89)
-		(diameter 0)
-		(color 0 0 0 0)
-	)
-	(junction
 		(at 200.66 121.92)
 		(diameter 0)
@@
 		)
 	)
-	(label "IO13"
+	(label "+3.3V"
 		(at 76.2 63.5 0)
 		(effects
@@
 		)
 	)
+	(label "GND"
+		(at 76.2 58.42 0)
+		(effects
+			(font
+				(size 1.27 1.27)
+			)
+			(justify left bottom)
+		)
+	)
+	(label "GND"
+		(at 76.2 68.58 0)
+		(effects
+			(font
+				(size 1.27 1.27)
+			)
+			(justify left bottom)
+		)
+	)
+	(label "+3.3V"
+		(at 76.2 53.34 0)
+		(effects
+			(font
+				(size 1.27 1.27)
+			)
+			(justify left bottom)
+		)
+	)
 	(label "EN"
 		(at 143.51 49.53 0)
@@
 		)
 	)
+	(label "GND"
+		(at 76.2 48.26 0)
+		(effects
+			(font
+				(size 1.27 1.27)
+			)
+			(justify left bottom)
+		)
+	)
 	(label "RX0"
 		(at 41.91 120.65 180)
@@
 	(label "IO0"
 		(at 236.22 148.59 0)
+		(effects
+			(font
+				(size 1.27 1.27)
+			)
+			(justify left bottom)
+		)
+	)
+	(label "+3.3V"
+		(at 76.2 43.18 0)
 		(effects
 			(font
@@
 	)
 	(symbol
-		(lib_id "Connector:USB_B_Mini")
-		(at 144.78 125.73 0)
-		(mirror y)
-		(unit 1)
-		(exclude_from_sim no)
-		(in_bom yes)
-		(on_board yes)
-		(dnp no)
-		(property "Reference" "J2"
-			(at 144.78 113.03 0)
-			(effects
-				(font
-					(size 1.27 1.27)
-				)
-			)
-		)
-		(property "Value" "USB_B_Mini"
-			(at 144.78 115.57 0)
-			(effects
-				(font
-					(size 1.27 1.27)
-				)
-			)
-		)
-		(property "Footprint" "User_Footprint:Usb_B_mini_Wurth_65100516121"
-			(at 140.97 127 0)
-			(effects
-				(font
-					(size 1.27 1.27)
-				)
-				(hide yes)
-			)
-		)
-		(property "Datasheet" "~"
-			(at 140.97 127 0)
-			(effects
-				(font
-					(size 1.27 1.27)
-				)
-				(hide yes)
-			)
-		)
-		(property "Description" "USB Mini Type B connector"
-			(at 144.78 125.73 0)
-			(effects
-				(font
-					(size 1.27 1.27)
-				)
-				(hide yes)
-			)
-		)
-		(pin "1"
-		)
-		(pin "3"
-		)
-		(pin "5"
-		)
-		(pin "2"
-		)
-		(pin "6"
-		)
-		(pin "4"
-		)
-		(instances
-			(project "esp-wroom-2-carrier-board"
-				(path "/02e826db-efcd-428f-8d48-cef0de8c3fb5/74f3df9c-3c45-447b-96d6-ab37cb14244d"
-					(reference "J2")
-					(unit 1)
-				)
-			)
-		)
-	)
-	(symbol
 		(lib_id "Device:R_US")
 		(at 208.28 139.7 90)
@@
 					(unit 1)
 				)
+			)
+		)
+	)
+	(symbol
+		(lib_id "Connector:USB_B_Mini")
+		(at 144.78 125.73 0)
+		(mirror y)
+		(unit 1)
+		(exclude_from_sim no)
+		(in_bom yes)
+		(on_board yes)
+		(dnp no)
+		(property "Reference" "J3"
+			(at 144.78 113.03 0)
+			(effects
+				(font
+					(size 1.27 1.27)
+				)
+			)
+		)
+		(property "Value" "USB_B_Mini"
+			(at 144.78 115.57 0)
+			(effects
+				(font
+					(size 1.27 1.27)
+				)
+			)
+		)
+		(property "Footprint" "Connector_USB:USB_Mini-B_Lumberg_2486_01_Horizontal"
+			(at 140.97 127 0)
+			(effects
+				(font
+					(size 1.27 1.27)
+				)
+				(hide yes)
+			)
+		)
+		(property "Datasheet" "~"
+			(at 140.97 127 0)
+			(effects
+				(font
+					(size 1.27 1.27)
+				)
+				(hide yes)
+			)
+		)
+		(property "Description" "USB Mini Type B connector"
+			(at 144.78 125.73 0)
+			(effects
+				(font
+					(size 1.27 1.27)
+				)
+				(hide yes)
+			)
+		)
+		(pin "5"
+		)
+		(pin "4"
+		)
+		(pin "3"
+		)
+		(pin "1"
+		)
+		(pin "6"
+		)
+		(pin "2"
+		)
+		(instances
+			(project ""
+				(path "/02e826db-efcd-428f-8d48-cef0de8c3fb5/74f3df9c-3c45-447b-96d6-ab37cb14244d"
+					(reference "J3")
+					(unit 1)
+				)

Commit message: capacitor layout
Changed capacitor position to front layer to have enough clearance on bottom layer
Parts:
- added TP1: 3.3V, TestPoint:TestPoint_THTPad_D1.0mm_Drill0.5mm, symbol Connector:TestPoint_Alt
- added TP3: GND, TestPoint:TestPoint_THTPad_D1.0mm_Drill0.5mm, symbol Connector:TestPoint_Alt
Connections:
- net +3.3V: now also TP1.1; no longer J1.5, J1.9
- net GND: now also TP3.1
- net VIN: now also J1.5, J1.9
Changed lines of the file:
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@@
 	)
 	(junction
+		(at 160.02 81.28)
+		(diameter 0)
+		(color 0 0 0 0)
+	)
+	(junction
 		(at 93.98 120.65)
 		(diameter 0)
@@
 	)
 	(junction
+		(at 82.55 43.18)
+		(diameter 0)
+		(color 0 0 0 0)
+	)
+	(junction
 		(at 132.08 52.07)
 		(diameter 0)
@@
 	)
 	(junction
+		(at 160.02 38.1)
+		(diameter 0)
+		(color 0 0 0 0)
+	)
+	(junction
 		(at 67.31 158.75)
 		(diameter 0)
@@
 	(wire
 		(pts
+			(xy 82.55 43.18) (xy 85.09 43.18)
+		)
+		(stroke
+			(width 0)
+			(type default)
+		)
+	)
+	(wire
+		(pts
 			(xy 67.31 76.2) (xy 76.2 76.2)
 		)
@@
 	(wire
 		(pts
-			(xy 160.02 74.93) (xy 160.02 78.74)
+			(xy 160.02 74.93) (xy 160.02 81.28)
 		)
 		(stroke
@@
 	(wire
 		(pts
+			(xy 160.02 81.28) (xy 167.64 81.28)
+		)
+		(stroke
+			(width 0)
+			(type default)
+		)
+	)
+	(wire
+		(pts
 			(xy 67.31 48.26) (xy 76.2 48.26)
 		)
@@
 	(wire
 		(pts
+			(xy 160.02 81.28) (xy 160.02 85.09)
+		)
+		(stroke
+			(width 0)
+			(type default)
+		)
+	)
+	(wire
+		(pts
 			(xy 64.77 100.33) (xy 93.98 100.33)
 		)
@@
 	(wire
 		(pts
-			(xy 67.31 53.34) (xy 76.2 53.34)
+			(xy 67.31 53.34) (xy 82.55 53.34)
 		)
 		(stroke
@@
 	(wire
 		(pts
+			(xy 82.55 53.34) (xy 82.55 43.18)
+		)
+		(stroke
+			(width 0)
+			(type default)
+		)
+	)
+	(wire
+		(pts
 			(xy 104.14 130.81) (xy 110.49 130.81)
 		)
@@
 	(wire
 		(pts
-			(xy 67.31 43.18) (xy 76.2 43.18)
+			(xy 67.31 43.18) (xy 82.55 43.18)
 		)
 		(stroke
@@
 		)
 	)
-	(label "+3.3V"
-		(at 76.2 53.34 0)
-		(effects
-			(font
-				(size 1.27 1.27)
-			)
-			(justify left bottom)
-		)
-	)
 	(label "EN"
 		(at 143.51 49.53 0)
@@
 		)
 	)
-	(label "+3.3V"
-		(at 76.2 43.18 0)
-		(effects
-			(font
-				(size 1.27 1.27)
-			)
-			(justify left bottom)
-		)
-	)
 	(label "IO4"
 		(at 179.07 54.61 0)
@@
 	(hierarchical_label "VIN"
 		(shape input)
-		(at 95.25 30.48 0)
+		(at 85.09 43.18 0)
 		(effects
 			(font
@@
 	)
 	(symbol
-		(lib_id "power:PWR_FLAG")
-		(at 71.12 27.94 0)
-		(unit 1)
-		(exclude_from_sim no)
-		(in_bom yes)
-		(on_board yes)
-		(dnp no)
-		(fields_autoplaced yes)
-		(property "Reference" "#FLG01"
-			(at 71.12 26.035 0)
-			(effects
-				(font
-					(size 1.27 1.27)
-				)
-				(hide yes)
-			)
-		)
-		(property "Value" "PWR_FLAG"
-			(at 71.12 22.86 0)
-			(effects
-				(font
-					(size 1.27 1.27)
-				)
-			)
-		)
-		(property "Footprint" ""
-			(at 71.12 27.94 0)
-			(effects
-				(font
-					(size 1.27 1.27)
-				)
-				(hide yes)
-			)
-		)
-		(property "Datasheet" "~"
-			(at 71.12 27.94 0)
-			(effects
-				(font
-					(size 1.27 1.27)
-				)
-				(hide yes)
-			)
-		)
-		(property "Description" "Special symbol for telling ERC where power comes from"
-			(at 71.12 27.94 0)
-			(effects
-				(font
-					(size 1.27 1.27)
-				)
-				(hide yes)
-			)
-		)
-		(pin "1"
-		)
-		(instances
-			(project ""
-				(path "/02e826db-efcd-428f-8d48-cef0de8c3fb5/74f3df9c-3c45-447b-96d6-ab37cb14244d"
-					(reference "#FLG01")
-					(unit 1)
-				)
-			)
-		)
-	)
-	(symbol
 		(lib_id "_Connectors:DF9B-19S-1V69")
 		(at 67.31 33.02 0)
@@
 	)
 	(symbol
+		(lib_id "Connector:TestPoint_Alt")
+		(at 160.02 38.1 0)
+		(unit 1)
+		(exclude_from_sim no)
+		(in_bom yes)
+		(on_board yes)
+		(dnp no)
+		(fields_autoplaced yes)
+		(property "Reference" "TP1"
+			(at 162.56 33.528 0)
+			(effects
+				(font
+					(size 1.27 1.27)
+				)
+				(justify left)
+			)
+		)
+		(property "Value" "3.3V"
+			(at 162.56 36.068 0)
+			(effects
+				(font
+					(size 1.27 1.27)
+				)
+				(justify left)
+			)
+		)
+		(property "Footprint" "TestPoint:TestPoint_THTPad_D1.0mm_Drill0.5mm"
+			(at 165.1 38.1 0)
+			(effects
+				(font
+					(size 1.27 1.27)
+				)
+				(hide yes)
+			)
+		)
+		(property "Datasheet" "~"
+			(at 165.1 38.1 0)
+			(effects
+				(font
+					(size 1.27 1.27)
+				)
+				(hide yes)
+			)
+		)
+		(property "Description" "test point (alternative shape)"
+			(at 160.02 38.1 0)
+			(effects
+				(font
+					(size 1.27 1.27)
+				)
+				(hide yes)
+			)
+		)
+		(pin "1"
+		)
+		(instances
+			(project ""
+				(path "/02e826db-efcd-428f-8d48-cef0de8c3fb5/74f3df9c-3c45-447b-96d6-ab37cb14244d"
+					(reference "TP1")
+					(unit 1)
+				)
+			)
+		)
+	)
+	(symbol
 		(lib_id "power:GND")
 		(at 144.78 140.97 0)
@@
 	(symbol
 		(lib_id "power:GND")
-		(at 160.02 78.74 0)
+		(at 160.02 85.09 0)
 		(unit 1)
 		(exclude_from_sim no)
@@
 		(fields_autoplaced yes)
 		(property "Reference" "#PWR09"
-			(at 160.02 85.09 0)
+			(at 160.02 91.44 0)
 			(effects
 				(font
@@
 		)
 		(property "Value" "GND"
-			(at 160.02 83.82 0)
+			(at 160.02 90.17 0)
 			(effects
 				(font
@@
 		)
 		(property "Footprint" ""
-			(at 160.02 78.74 0)
+			(at 160.02 85.09 0)
 			(effects
 				(font
@@
 		)
 		(property "Datasheet" ""
-			(at 160.02 78.74 0)
+			(at 160.02 85.09 0)
 			(effects
 				(font
@@
 		)
 		(property "Description" "Power symbol creates a global label with name \"GND\" , ground"
-			(at 160.02 78.74 0)
+			(at 160.02 85.09 0)
 			(effects
 				(font
@@
 					(unit 1)
 				)
+			)
+		)
+	)
+	(symbol
+		(lib_id "Connector:TestPoint_Alt")
+		(at 167.64 81.28 0)
+		(unit 1)
+		(exclude_from_sim no)
+		(in_bom yes)
+		(on_board yes)
+		(dnp no)
+		(fields_autoplaced yes)
+		(property "Reference" "TP3"
+			(at 170.18 76.708 0)
+			(effects
+				(font
+					(size 1.27 1.27)
+				)
+				(justify left)
+			)
+		)
+		(property "Value" "GND"
+			(at 170.18 79.248 0)
+			(effects
+				(font
+					(size 1.27 1.27)
+				)
+				(justify left)
+			)
+		)
+		(property "Footprint" "TestPoint:TestPoint_THTPad_D1.0mm_Drill0.5mm"
+			(at 172.72 81.28 0)
+			(effects
+				(font
+					(size 1.27 1.27)
+				)
+				(hide yes)
+			)
+		)
+		(property "Datasheet" "~"
+			(at 172.72 81.28 0)
+			(effects
+				(font
+					(size 1.27 1.27)
+				)
+				(hide yes)
+			)
+		)
+		(property "Description" "test point (alternative shape)"
+			(at 167.64 81.28 0)
+			(effects
+				(font
+					(size 1.27 1.27)
+				)
+				(hide yes)
+			)
+		)
+		(pin "1"
+		)
+		(instances
+			(project "esp-wroom-2-carrier-board"
+				(path "/02e826db-efcd-428f-8d48-cef0de8c3fb5/74f3df9c-3c45-447b-96d6-ab37cb14244d"
+					(reference "TP3")
+					(unit 1)
+				)
