File: Stm/stm32g431kb-som/stm32g431/stm32g431.kicad_sch (KiCad schematic)
At the start: 3 parts, among them J1 Conn_ARM_JTAG_SWD_10, U1 STM32G431KBTx, m1 M.2-B+M-KEY

Commit message: PCB
Create pcb
Parts:
- removed m1: M.2-B+M-KEY, User_Footprint:M.2-B-KEY, symbol _Connectors:M.2-B+M-KEY
- added C1: ~, User_Footprint:Mini PCI express Half, symbol Cards:Mini_PCIexpress_Half
- added Y1: ECS-TXO-3225-250-TR, User_Footprint:OSC_ECS-TXO-3225-250-TR, symbol _Misc_Symborls:ECS-TXO-3225-250-TR
Connections:
- net GND: now also C1.2, C1.4, C1.6, C1.8
- net PA0: now also C1.13
- net PA1: now also C1.15
- net PA10: now also C1.33
- net PA11: now also C1.35
- net PA12: now also C1.37
- net PA15: now also C1.43
- net PA2: now also C1.17
- net PA3: now also C1.19
- net PA4: now also C1.21
- net PA5: now also C1.23
- net PA6: now also C1.25
- net PA7: now also C1.27
- net PA8: now also C1.29
- net PA9: now also C1.31
- net PB0: now also C1.14
- net PB3: now also C1.16
- net PB4: now also C1.18
- net PB5: now also C1.20
- net PB6: now also C1.22
- net PB7: now also C1.24
- net PB8: now also C1.26
- net VDD: now also C1.1, C1.3, C1.5
- net VDDA: now also C1.7
- new net +3.3V: Y1.4 (VDD)
- new net PA13: C1.39
- new net PA14: C1.41
- no-connect marks 0 -> 1

Commit message: Pcb
Add more components
Parts:
- removed Y1: ECS-TXO-3225-250-TR, User_Footprint:OSC_ECS-TXO-3225-250-TR, symbol _Misc_Symborls:ECS-TXO-3225-250-TR
- added C2, C3: C, Capacitor_SMD:C_01005_0402Metric, symbol Device:C
- added C4: 22uF, symbol Device:C_Polarized_US
- added C5: 15uF, symbol Device:C_Polarized_US
- added D1, D3: BAT60A, Diode_SMD:D_SOD-323, symbol Diode:BAT60A
- added J2: USB_C_Receptacle_USB2.0_16P, Connector_USB:USB_C_Receptacle_G-Switch_GT-USB-7010ASV, symbol Connector:USB_C_Receptacle_USB2.0_16P
- added R1, R2, R3, R4, R5, R6, R7: 0, Resistor_SMD:R_01005_0402Metric, symbol Device:R_US
- added U3: LD1117S33TR_SOT223, Package_TO_SOT_SMD:SOT-223-3_TabPin2, symbol Regulator_Linear:LD1117S33TR_SOT223
- added Y1: ECS-250-10-37B-CTN-TR, User_Footprint:XTAL_ECS-160-9-37-CKM-TR, symbol _Misc_Symborls:ECS-250-10-37B-CTN-TR
Connections:
- net GND: now also C2.2, C3.2, C4.2, C5.2, J2.A1 (GND), J2.A12 (GND), J2.B1 (GND), J2.B12 (GND), J2.S1 (SHIELD), U3.1 (GND), Y1.2 (GND), Y1.4 (GND__1)
- net PA11: now also R6.2
- net PA12: now also R7.2
- net VDD: now also D3.2 (A); no longer U1.1 (VDD), U1.17 (VDD)
- net VDDA: now also U1.15 (VDDA)
- net PF0: now reaches U1.2 (PF0)
- net PF0: now also R1.2, R2.2
- net PF1: now reaches U1.3 (PF1)
- net PF1: now also R3.2, R4.2
- net PG10: now reaches U1.4 (PG10)
- net PG10: now also C1.9
- net +3V3: now reaches J1.1 (VTref)
- net +3V3: now also U1.1 (VDD), U1.17 (VDD), R5.2
- net at C1.10: now also R2.1
- net at C1.12: now also R4.1
- new net: C4.1, R5.1, U3.2 (VO)
- new net: C5.1, D1.1 (K), D3.1 (K), U3.3 (VI)
- new net: D1.2 (A), J2.A4 (VBUS), J2.A9 (VBUS), J2.B4 (VBUS), J2.B9 (VBUS)
- new net DM: J2.A7 (D-), J2.B7 (D-), R6.1
- new net DP: J2.A6 (D+), J2.B6 (D+), R7.1
- new net OSC_IN: C2.1, R1.1, Y1.3 (OUT/IN)
- new net OSC_OUT: C3.1, R3.1, Y1.1 (IN/OUT)
- no-connect marks 1 -> 6

Commit message: SOM
Added Card Holes, Needed?
Parts:
- removed D1, D3: BAT60A, Diode_SMD:D_SOD-323, symbol Diode:BAT60A
- removed U3: LD1117S33TR_SOT223, Package_TO_SOT_SMD:SOT-223-3_TabPin2, symbol Regulator_Linear:LD1117S33TR_SOT223
- removed Y1: ECS-250-10-37B-CTN-TR, User_Footprint:XTAL_ECS-160-9-37-CKM-TR, symbol _Misc_Symborls:ECS-250-10-37B-CTN-TR
- added D1: BAT54CW, Package_TO_SOT_SMD:SOT-323_SC-70, symbol Diode:BAT54CW
- added H1, H3: MountingHole_Pad, MountingHole:MountingHole_2.2mm_M2_DIN965_Pad, symbol Mechanical:MountingHole_Pad
- added U2: AP7361C-33E, Package_TO_SOT_SMD:SOT-223-3_TabPin2, symbol Regulator_Linear:AP7361C-33E
- added Y2: 24Mhz, User_Footprint:jxs11, symbol _Misc_Symbols:JXS11-12-10/10
- C4, C5: footprint (none) -> Capacitor_Tantalum_SMD:CP_EIA-7343-30_AVX-N
Connections:
- net GND: now also U2.2 (GND), Y2.2 (GND), Y2.4 (GND)
- net OSC_IN: now also Y2.3
- net OSC_OUT: now also Y2.1
- net VDD: now also D1.2
- net at C4.1, R5.1: now also U2.3 (VO)
- net at C5.1: now also D1.3, U2.1 (VI)
- net at J2.A4 (VBUS), J2.A9 (VBUS), J2.B4 (VBUS)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: now also D1.1
Other:
- moved on the sheet: C2, R1

Commit message: Pcb
Pre-final PCB
Parts:
- removed C4: 22uF, Capacitor_Tantalum_SMD:CP_EIA-7343-30_AVX-N, symbol Device:C_Polarized_US
- removed C5: 15uF, Capacitor_Tantalum_SMD:CP_EIA-7343-30_AVX-N, symbol Device:C_Polarized_US
- removed H1, H3: MountingHole_Pad, MountingHole:MountingHole_2.2mm_M2_DIN965_Pad, symbol Mechanical:MountingHole_Pad
- added C10, C9: 1uF, Capacitor_SMD:C_01005_0402Metric, symbol Device:C
- added C4: 1uF, Capacitor_SMD:C_0805_2012Metric, symbol Device:C
- added C5: 4.7uF, Capacitor_SMD:C_0805_2012Metric, symbol Device:C
- added C6: 100nF, Capacitor_SMD:C_0402_1005Metric, symbol Device:C
- added C7, C8: 100nF, Capacitor_SMD:C_01005_0402Metric, symbol Device:C
- added D2, D3: PGB1010603NR, User_Footprint:DIOC1608X36N, symbol _Misc_Symbols:PGB1010603NR
- added D4: LED, LED_SMD:LED_0402_1005Metric, symbol Device:LED
- added R8: 0, Resistor_SMD:R_01005_0402Metric, symbol Device:R_US
- added R9: 100, Resistor_SMD:R_01005_0402Metric, symbol Device:R_US
- added S1: 436331045822, User_Footprint:4363X10458XX, symbol _Misc_Symbols:436331045822
- J2: footprint Connector_USB:USB_C_Receptacle_G-Switch_GT-USB-7010ASV -> User_Footprint:AMPHENOL_GSB1C41110SSHR; symbol Connector:USB_C_Receptacle_USB2.0_16P -> _Connectors:GSB1C41110SSHR; MANUFACTURER (none) -> Amphenol; MAXIMUM_PACKAGE_HEIGHT (none) -> 3.21mm; PARTREV (none) -> AX1; STANDARD (none) -> Manufacturer Recommendations
- R5: footprint Resistor_SMD:R_01005_0402Metric -> Resistor_SMD:R_0805_2012Metric
Connections:
- net PA13 is gone; now on net PA5: C1.39
- net PA14 is gone; now on net PA6: C1.41
- net +3V3: now also C10.1, C7.1, C8.1, C9.1, R9.2
- net DM: now also D3.2
- net DP: now also D2.1
- net GND: now also C1.51, J2.A1_B12 (GND), J2.B1_A12 (GND), J2.SH1 (SHIELD), C10.2, C4.2, C5.2, C6.2, C7.2, C8.2, C9.2, D2.2, D3.1, D4.1 (K), S1.2, S1.4; no longer J2.A1 (GND), J2.A12 (GND), J2.B1 (GND), J2.B12 (GND), J2.S1 (SHIELD)
- net PA0: now also C1.29; no longer C1.13
- net PA1: now also C1.31; no longer C1.15
- net PA10: now also C1.48; no longer C1.33
- net PA11: now also C1.46; no longer C1.35
- net PA12: now also C1.44; no longer C1.37
- net PA15: now also C1.42; no longer C1.43
- net PA2: now also C1.33; no longer C1.17
- net PA3: now also C1.35; no longer C1.19
- net PA4: now also C1.37; no longer C1.21
- net PA5: no longer C1.23
- net PA6: no longer C1.25
- net PA7: now also C1.43; no longer C1.27
- net PA8: now also C1.52; no longer C1.29
- net PA9: now also C1.50; no longer C1.31
- net PB0: now also C1.45; no longer C1.14
- net PB3: now also C1.40; no longer C1.16
- net PB4: now also C1.38; no longer C1.18
- net PB5: now also C1.36; no longer C1.20
- net PB6: now also C1.34; no longer C1.22
- net PB7: now also C1.32; no longer C1.24
- net PB8: now also C1.30; no longer C1.26
- net PF1: now also R4.1; no longer R4.2
- net PG10: now also C1.27, R8.2; no longer C1.9
- net VDDA: now also C1.47, C1.49; no longer C1.7
- net at R5.1, U2.3 (VO): now also C5.1
- net at D1.3, U2.1 (VI): now also C4.1
- net at C1.12: no longer R4.1
- net at C1.10: no longer R2.1
- net PFR0: now reaches C1.28
- net PFR0: now also R2.1
- new net: C6.1, R8.1, S1.1, S1.3
- new net: D4.2 (A), R9.1
- new net PFR1: C1.26, R4.2
- new net VBUS: D1.1, J2.A4_B9 (VBUS), J2.B4_A9 (VBUS)
- no-connect marks 6 -> 7
Other:
- moved on the sheet: J2, R2, R4, R6, R7
