File: Stm/driverModule/tranceivers.kicad_sch (KiCad schematic)
At the start: 12 parts, among them U103 TJA1051T-3, U3 MCP2003B-E/SN

Commit message: Connectors
Remove some enable signals
Added Harness connectors
Parts:
- added R12: 10K, Resistor_SMD:R_0402_1005Metric, symbol Device:R_US
- C1, C2: footprint (none) -> Capacitor_SMD:C_0402_1005Metric
Connections:
- net GND: now also R12.2
- net CANSilentMode: no longer names the net of U103.8 (S)
- net CANSilentMode: now also R12.1
