File: Stm/driverModule/Power.kicad_sch (KiCad schematic)
At the start: 12 parts, among them U102 ADM7171ACPZ-3.0-R7, U104 TPS5410DR

Commit message: routing
Finished PCB routing
Parts:
- added TP1, TP2, TP3: TestPoint_Small, TestPoint:TestPoint_Pad_1.0x1.0mm, symbol Connector:TestPoint_Small
Connections:
- net +12V: now also TP3.1
- net +3V3: now also TP1.1
- net +5V: now also TP2.1
