File: misc/Pcie_Breakout_Board/pcieBreakOutBoard/Power3v3.kicad_sch (KiCad schematic)
At the start: 12 parts, among them J2 USB_C_Receptacle_USB2.0_16P, U2 AP7361C-33E

Commit message: Jtag
Added jtag and serial interface to the breakout board
Connections:
- net VBUS renamed Vbus
Changed lines of the file:
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@@
+	)
+	(junction
+		(at 135.89 77.47)
+		(diameter 0)
+		(color 0 0 0 0)
 	)
 	(junction
@@
 	(wire
 		(pts
+			(xy 135.89 63.5) (xy 135.89 77.47)
+		)
+		(stroke
+			(width 0)
+			(type default)
+		)
+	)
+	(wire
+		(pts
 			(xy 209.55 96.52) (xy 209.55 99.06)
 		)
@@
 	(wire
 		(pts
-			(xy 123.19 77.47) (xy 144.78 77.47)
+			(xy 123.19 77.47) (xy 135.89 77.47)
 		)
 		(stroke
@@
 	(wire
 		(pts
+			(xy 135.89 77.47) (xy 144.78 77.47)
+		)
+		(stroke
+			(width 0)
+			(type default)
+		)
+	)
+	(wire
+		(pts
 			(xy 132.08 110.49) (xy 134.62 110.49)
 		)
@@
 			(width 0)
 			(type default)
-		)
-	)
-	(label "VBUS"
-		(at 128.27 77.47 0)
-		(effects
-			(font
-				(size 1.27 1.27)
-			)
-			(justify left bottom)
 		)
 	)
@@
 		)
 	)
+	(hierarchical_label "Vbus"
+		(shape output)
+		(at 135.89 63.5 0)
+		(effects
+			(font
+				(size 1.27 1.27)
+			)
+			(justify left)
+		)
+	)
