File: misc/Pcie_Breakout_Board/pcieBreakOutBoard/MiniPcieExHalf.kicad_sch (KiCad schematic)
At the start: 1 part, among them J3 2041119-1 (Mini Pcie Express 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

Commit message: layout
finished 70% of layout
Parts:
- J3: footprint User_Footprint:CONN_2041119-1_TEC -> Connector_PCBEdge:BUS_PCI_Express_Mini_Half
Changed lines of the file:
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@@
 			)
 		)
-		(property "Footprint" "User_Footprint:CONN_2041119-1_TEC"
+		(property "Footprint" "Connector_PCBEdge:BUS_PCI_Express_Mini_Half"
 			(at 147.574 60.706 0)
 			(effects
